Commit message: first commit

File: catkin_ws/src/my_robot/urdf/my_robot.xacro (robot description, xacro)
@@ -147,4 +147,11 @@
     </intertial>
  </link>
+<joint name="camera_optical_joint" type="fixed">
+    <origin xyz="0 0 0" rpy="-1.5707 0 -1.5707"/>
+    <parent link="camera_link"/>
+    <child link="camera_link_optical"/>
+  </joint>
+  <link name="camera_link_optical">
+  </link>
  <joint type="fixed" name="hokuyo_joint">
     <origin xyz="0.15 0 0.1" rpy="0 0 0"/>

Commit message: first commit

File: catkin_ws/src/my_robot/urdf/my_robot.xacro (robot description, xacro)
@@ -147,7 +147,8 @@
     </intertial>
  </link>
-<joint name="camera_optical_joint" type="fixed">
+  <!-- <link name="camera_link" /> -->
+  <joint name="camera_optical_joint" type="fixed">
     <origin xyz="0 0 0" rpy="-1.5707 0 -1.5707"/>
-    <parent link="camera_link"/>
+    <parent link="camera"/>
     <child link="camera_link_optical"/>
   </joint>
